File: AX12/ax12.sch (EAGLE design)
At the start: 14 parts

Commit message: fix board et gerber file
Parts:
- removed 74HC126-1, 74HC126-2: (no value), con-lstb:MA07-1
- added IC1: (no value), ic-package:DIL14
Connections:
- net 5V: now also IC1.14; no longer 74HC126-1.7
- net AX12-DATA: now also IC1.12; no longer 74HC126-1.5
- net GND: now also IC1.7; no longer 74HC126-2.7
- net RXD: now also IC1.11; no longer 74HC126-1.4
- net TXD: now also IC1.13; no longer 74HC126-1.6
Changed lines of the file:
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@@
 <parts>
 <part name="FRAME1" library="frames" library_urn="urn:adsk.eagle:library:229" deviceset="A4L-LOC" device=""/>
-<part name="74HC126-1" library="con-lstb" library_urn="urn:adsk.eagle:library:162" deviceset="MA07-1" device="" package3d_urn="urn:adsk.eagle:package:8341/1"/>
-<part name="74HC126-2" library="con-lstb" library_urn="urn:adsk.eagle:library:162" deviceset="MA07-1" device="" package3d_urn="urn:adsk.eagle:package:8341/1"/>
 <part name="FTDI-1" library="con-lstb" library_urn="urn:adsk.eagle:library:162" deviceset="MA09-1" device="" package3d_urn="urn:adsk.eagle:package:8350/1"/>
 <part name="FTDI-2" library="con-lstb" library_urn="urn:adsk.eagle:library:162" deviceset="MA09-1" device="" package3d_urn="urn:adsk.eagle:package:8350/1"/>
@@
 <part name="ALIM-AX12-3" library="con-molex" library_urn="urn:adsk.eagle:library:165" deviceset="22-23-2021" device=""/>
 <part name="ALIM-AX12-4" library="con-molex" library_urn="urn:adsk.eagle:library:165" deviceset="22-23-2021" device=""/>
+<part name="IC1" library="ic-package" library_urn="urn:adsk.eagle:library:239" deviceset="DIL14" device="" package3d_urn="urn:adsk.eagle:package:16407/2"/>
 </parts>
 <sheets>
@@
 <attribute name="LAST_DATE_TIME" x="97.79" y="-78.74" size="2.286" layer="94"/>
 <attribute name="SHEET" x="111.125" y="-83.82" size="2.54" layer="94"/>
-</instance>
-<instance part="74HC126-1" gate="1" x="2.54" y="-2.54" smashed="yes" rot="R90">
-<attribute name="VALUE" x="15.24" y="-3.81" size="1.778" layer="96" rot="R90"/>
-<attribute name="NAME" x="-8.382" y="-3.81" size="1.778" layer="95" rot="R90"/>
-</instance>
-<instance part="74HC126-2" gate="1" x="2.54" y="-10.16" smashed="yes" rot="R270">
-<attribute name="VALUE" x="-10.16" y="-8.89" size="1.778" layer="96" rot="R270"/>
-<attribute name="NAME" x="13.462" y="-8.89" size="1.778" layer="95" rot="R270"/>
 </instance>
 <instance part="FTDI-1" gate="1" x="-50.8" y="-7.62" smashed="yes">
@@
 <attribute name="NAME" x="88.138" y="17.78" size="1.524" layer="95" rot="R270"/>
 </instance>
+<instance part="IC1" gate="G$1" x="2.54" y="-7.62" smashed="yes" rot="R90">
+<attribute name="NAME" x="-6.985" y="-12.065" size="1.778" layer="95" rot="R90"/>
+<attribute name="VALUE" x="13.97" y="-12.065" size="1.778" layer="96" rot="R90"/>
+</instance>
 </instances>
 <busses>
@@
 <net name="5V" class="0">
 <segment>
-<pinref part="74HC126-1" gate="1" pin="7"/>
-<wire x1="-5.08" y1="5.08" x2="-5.08" y2="12.7" width="0.1524" layer="91"/>
+<wire x1="-5.08" y1="0" x2="-5.08" y2="12.7" width="0.1524" layer="91"/>
 <pinref part="R1" gate="G$1" pin="1"/>
 <wire x1="-5.08" y1="12.7" x2="-5.08" y2="15.24" width="0.1524" layer="91"/>
@@
 <wire x1="-68.58" y1="-10.16" x2="-78.74" y2="-10.16" width="0.1524" layer="91"/>
 <wire x1="-78.74" y1="12.7" x2="-78.74" y2="-10.16" width="0.1524" layer="91"/>
+<pinref part="IC1" gate="G$1" pin="14"/>
 </segment>
 </net>
@@
 <pinref part="FTDI-1" gate="1" pin="7"/>
 <wire x1="-43.18" y1="-2.54" x2="-17.78" y2="-2.54" width="0.1524" layer="91"/>
-<pinref part="74HC126-2" gate="1" pin="7"/>
-<wire x1="10.16" y1="-17.78" x2="10.16" y2="-22.86" width="0.1524" layer="91"/>
+<wire x1="10.16" y1="-15.24" x2="10.16" y2="-22.86" width="0.1524" layer="91"/>
 <wire x1="-17.78" y1="-2.54" x2="-17.78" y2="-22.86" width="0.1524" layer="91"/>
 <wire x1="-17.78" y1="-22.86" x2="10.16" y2="-22.86" width="0.1524" layer="91"/>
@@
 <wire x1="91.44" y1="22.86" x2="91.44" y2="33.02" width="0.1524" layer="91"/>
 <junction x="91.44" y="33.02"/>
+<pinref part="IC1" gate="G$1" pin="7"/>
 </segment>
 </net>
 <net name="TXD" class="0">
 <segment>
-<pinref part="74HC126-1" gate="1" pin="6"/>
-<wire x1="-2.54" y1="5.08" x2="-2.54" y2="12.7" width="0.1524" layer="91"/>
+<wire x1="-2.54" y1="0" x2="-2.54" y2="12.7" width="0.1524" layer="91"/>
 <pinref part="D1" gate="1" pin="C"/>
 <junction x="-2.54" y="12.7"/>
@@
 <wire x1="-2.54" y1="27.94" x2="-38.1" y2="27.94" width="0.1524" layer="91"/>
 <wire x1="-38.1" y1="27.94" x2="-38.1" y2="-17.78" width="0.1524" layer="91"/>
+<pinref part="IC1" gate="G$1" pin="13"/>
 </segment>
 </net>
@@
 <segment>
 <pinref part="FTDI-1" gate="1" pin="5"/>
-<pinref part="74HC126-1" gate="1" pin="4"/>
-<wire x1="2.54" y1="5.08" x2="2.54" y2="-7.62" width="0.1524" layer="91"/>
 <wire x1="2.54" y1="-7.62" x2="-43.18" y2="-7.62" width="0.1524" layer="91"/>
+<pinref part="IC1" gate="G$1" pin="11"/>
+<wire x1="2.54" y1="0" x2="2.54" y2="-7.62" width="0.1524" layer="91"/>
 </segment>
 </net>
 <net name="AX12-DATA" class="0">
 <segment>
-<pinref part="74HC126-1" gate="1" pin="5"/>
-<wire x1="0" y1="5.08" x2="0" y2="7.62" width="0.1524" layer="91"/>
 <wire x1="0" y1="7.62" x2="2.54" y2="7.62" width="0.1524" layer="91"/>
 <pinref part="D1" gate="1" pin="A"/>
@@
 <pinref part="AX12-4" gate="G$1" pin="1"/>
 <wire x1="86.36" y1="35.56" x2="86.36" y2="38.1" width="0.1524" layer="91"/>
+<pinref part="IC1" gate="G$1" pin="12"/>
+<wire x1="0" y1="7.62" x2="0" y2="0" width="0.1524" layer="91"/>
 </segment>
 </net>
