File: Asserv v2/asserv v2.brd (EAGLE design)
At the start: 81.3 x 64.4 mm, 6 parts, among them U1 NUCLEO-F446RE

Commit message: maj asserv nucelo
Parts:
- removed ALIM: 22-23-2021, con-molex:22-23-2021
- added BATTERIE, RESET: 22-23-2021, con-molex:22-23-2021
- added C1: 0.33uF, capacitor-wima:C5B2.5
- added C2: 0.1uF, capacitor-wima:C5B2.5
- added IC1: 7805TV, linear:TO220V
Connections:
- removed net AGND: U1.CN10_32
- removed net CN10_GND: U1.CN10_20, U1.CN10_9
- removed net CN5_GND: U1.CN5_7
- removed net CN6_GND: U1.CN6_6, U1.CN6_7
- removed net E5V: U1.CN7_6
- new net CN6_+5V: U1.CN6_5
- new net CN7_+5V: U1.CN7_18
- new net N$1: BATTERIE.2, C1.1, IC1.1
- new net N$4: RESET.2, U1.CN7_14
- net 5V: now also C2.1, IC1.3, U1.CN7_6; no longer ALIM.2, U1.CN6_5, U1.CN7_18
- net GND: now also BATTERIE.1, C1.2, C2.2, IC1.2, RESET.1, U1.CN10_20, U1.CN10_32, U1.CN10_9, U1.CN5_7, U1.CN6_6, U1.CN6_7; no longer ALIM.1
Routing:
- net N$4: track 0.00 -> 44.5 mm, vias 0 -> 2
- net 5V: track 90.7 -> 111.4 mm
- net N$1: track 0.00 -> 12.7 mm
- net GND: track 0.00 -> 5.08 mm, vias 0 -> 2

Commit message: gerber file for IA V2 + new libraries from mouser + Lidar / Ia / Asserv shield project creation
Parts:
- added R1, R2: (no value), rcl:0204/7
- turned USB to 180 degrees
Connections:
- net 5V: now also R1.2, R2.2
- net SCL: now also R2.1
- net SDA: now also R1.1
Routing:
- net 5V: track 111.4 -> 156.3 mm, vias 0 -> 2
- net D+: track 51.2 -> 58.1 mm
- net SCL: track 56.0 -> 59.4 mm
- net D-: track 64.3 -> 62.2 mm
- net N$4: track 44.5 -> 42.7 mm
- net SDA: track 65.1 -> 66.6 mm
Other:
- board size 81.3 x 64.4 mm -> 80 x 86 mm
