File: Asserv v2/asserv v2.sch (EAGLE design)
At the start: 6 parts, among them U1 NUCLEO-F446RE

Commit message: maj asserv nucelo
Parts:
- removed ALIM: 22-23-2021, con-molex:22-23-2021
- added BATTERIE, RESET: 22-23-2021, con-molex:22-23-2021
- added C1: 0.33uF, capacitor-wima:C5/2.5
- added C2: 0.1uF, capacitor-wima:C5/2.5
- added IC1: 7805TV, linear:7805TV
Connections:
- new net N$1: BATTERIE-2.S, C1.1, IC1.VI
- new net N$4: RESET-2.S, U1G$1.CN7_RESET
- net 5V: now also C2.1, IC1.VO, U1G$1.E5V; no longer ALIM-2.S, U1G$1.CN7_+5V, U1G$3.CN6_+5V
- net GND: now also BATTERIE-1.S, C1.2, C2.2, IC1.GND, RESET-1.S, U1G$2.AGND, U1G$2.CN10_GND, U1G$3.CN6_GND, U1G$6.CN5_GND; no longer ALIM-1.S
Changed lines of the file:
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@@
 <part name="CODEUR2" library="con-molex" library_urn="urn:adsk.eagle:library:165" deviceset="22-23-2041" device="" package3d_urn="urn:adsk.eagle:package:8078635/1"/>
 <part name="USB" library="con-lsta" library_urn="urn:adsk.eagle:library:161" deviceset="FE05-1" device="" package3d_urn="urn:adsk.eagle:package:8190/1"/>
-<part name="ALIM" library="con-molex" library_urn="urn:adsk.eagle:library:165" deviceset="22-23-2021" device="" package3d_urn="urn:adsk.eagle:package:8078633/1"/>
+<part name="IC1" library="linear" library_urn="urn:adsk.eagle:library:262" deviceset="78*" device="TV" technology="05"/>
+<part name="BATTERIE" library="con-molex" library_urn="urn:adsk.eagle:library:165" deviceset="22-23-2021" device=""/>
+<part name="C1" library="capacitor-wima" library_urn="urn:adsk.eagle:library:116" deviceset="C" device="5/2.5" value="0.33uF"/>
+<part name="C2" library="capacitor-wima" library_urn="urn:adsk.eagle:library:116" deviceset="C" device="5/2.5" value="0.1uF"/>
+<part name="RESET" library="con-molex" library_urn="urn:adsk.eagle:library:165" deviceset="22-23-2021" device=""/>
 </parts>
 <sheets>
@@
 <attribute name="NAME" x="19.05" y="99.822" size="1.778" layer="95"/>
 </instance>
-<instance part="ALIM" gate="-1" x="22.86" y="68.58" smashed="yes" rot="R180">
-<attribute name="NAME" x="20.32" y="69.342" size="1.524" layer="95" rot="R180"/>
-<attribute name="VALUE" x="23.622" y="67.183" size="1.778" layer="96" rot="R180"/>
-</instance>
-<instance part="ALIM" gate="-2" x="22.86" y="71.12" smashed="yes" rot="R180">
-<attribute name="NAME" x="20.32" y="71.882" size="1.524" layer="95" rot="R180"/>
-</instance>
 <instance part="U1" gate="G$3" x="218.44" y="58.42" smashed="yes">
 <attribute name="NAME" x="203.2" y="69.85" size="1.778" layer="95"/>
@@
 <attribute name="NAME" x="99.06" y="49.53" size="1.778" layer="95"/>
 <attribute name="VALUE" x="99.06" y="13.97" size="1.778" layer="96" rot="MR180"/>
+</instance>
+<instance part="IC1" gate="A1" x="45.72" y="60.96" smashed="yes">
+<attribute name="NAME" x="38.1" y="66.675" size="1.778" layer="95"/>
+<attribute name="VALUE" x="38.1" y="64.135" size="1.778" layer="96"/>
+</instance>
+<instance part="BATTERIE" gate="-1" x="20.32" y="58.42" smashed="yes" rot="R180">
+<attribute name="NAME" x="17.78" y="59.182" size="1.524" layer="95" rot="R180"/>
+<attribute name="VALUE" x="21.082" y="57.023" size="1.778" layer="96" rot="R180"/>
+</instance>
+<instance part="BATTERIE" gate="-2" x="20.32" y="60.96" smashed="yes" rot="R180">
+<attribute name="NAME" x="17.78" y="61.722" size="1.524" layer="95" rot="R180"/>
+</instance>
+<instance part="C1" gate="G$1" x="27.94" y="58.42" smashed="yes">
+<attribute name="NAME" x="29.464" y="58.801" size="1.778" layer="95"/>
+<attribute name="VALUE" x="29.464" y="53.721" size="1.778" layer="96"/>
+</instance>
+<instance part="C2" gate="G$1" x="63.5" y="58.42" smashed="yes">
+<attribute name="NAME" x="65.024" y="58.801" size="1.778" layer="95"/>
+<attribute name="VALUE" x="65.024" y="53.721" size="1.778" layer="96"/>
+</instance>
+<instance part="RESET" gate="-1" x="78.74" y="134.62" smashed="yes" rot="R180">
+<attribute name="NAME" x="76.2" y="135.382" size="1.524" layer="95" rot="R180"/>
+<attribute name="VALUE" x="79.502" y="133.223" size="1.778" layer="96" rot="R180"/>
+</instance>
+<instance part="RESET" gate="-2" x="78.74" y="137.16" smashed="yes" rot="R180">
+<attribute name="NAME" x="76.2" y="137.922" size="1.524" layer="95" rot="R180"/>
 </instance>
 </instances>
@@
 </segment>
 <segment>
-<pinref part="U1" gate="G$1" pin="CN7_+5V"/>
-<wire x1="152.4" y1="152.4" x2="162.56" y2="152.4" width="0.1524" layer="91"/>
-<label x="162.56" y="152.4" size="1.778" layer="95"/>
-</segment>
-<segment>
 <pinref part="CODEUR1" gate="-2" pin="S"/>
 <wire x1="27.94" y1="137.16" x2="40.64" y2="137.16" width="0.1524" layer="91"/>
@@
 </segment>
 <segment>
-<pinref part="ALIM" gate="-2" pin="S"/>
-<wire x1="25.4" y1="71.12" x2="40.64" y2="71.12" width="0.1524" layer="91"/>
-<label x="40.64" y="71.12" size="1.778" layer="95"/>
-</segment>
-<segment>
-<pinref part="U1" gate="G$3" pin="CN6_+5V"/>
-<wire x1="238.76" y1="63.5" x2="246.38" y2="63.5" width="0.1524" layer="91"/>
-<label x="246.38" y="63.5" size="1.778" layer="95"/>
+<pinref part="U1" gate="G$1" pin="E5V"/>
+<wire x1="152.4" y1="149.86" x2="162.56" y2="149.86" width="0.1524" layer="91"/>
+<label x="162.56" y="149.86" size="1.778" layer="95"/>
+</segment>
+<segment>
+<pinref part="IC1" gate="A1" pin="VO"/>
+<pinref part="C2" gate="G$1" pin="1"/>
+<wire x1="55.88" y1="60.96" x2="63.5" y2="60.96" width="0.1524" layer="91"/>
+<wire x1="73.66" y1="60.96" x2="63.5" y2="60.96" width="0.1524" layer="91"/>
+<junction x="63.5" y="60.96"/>
+<label x="73.66" y="60.96" size="1.778" layer="95"/>
 </segment>
 </net>
@@
 </segment>
 <segment>
-<pinref part="ALIM" gate="-1" pin="S"/>
-<wire x1="25.4" y1="68.58" x2="40.64" y2="68.58" width="0.1524" layer="91"/>
-<label x="40.64" y="68.58" size="1.778" layer="95"/>
+<pinref part="C1" gate="G$1" pin="2"/>
+<pinref part="IC1" gate="A1" pin="GND"/>
+<wire x1="27.94" y1="53.34" x2="45.72" y2="53.34" width="0.1524" layer="91"/>
+<pinref part="C2" gate="G$1" pin="2"/>
+<wire x1="45.72" y1="53.34" x2="63.5" y2="53.34" width="0.1524" layer="91"/>
+<junction x="45.72" y="53.34"/>
+<pinref part="BATTERIE" gate="-1" pin="S"/>
+<wire x1="22.86" y1="58.42" x2="22.86" y2="48.26" width="0.1524" layer="91"/>
+<wire x1="22.86" y1="48.26" x2="45.72" y2="48.26" width="0.1524" layer="91"/>
+<wire x1="45.72" y1="48.26" x2="45.72" y2="53.34" width="0.1524" layer="91"/>
+<junction x="45.72" y="48.26"/>
+<wire x1="45.72" y1="48.26" x2="45.72" y2="43.18" width="0.1524" layer="91"/>
+<label x="45.72" y="43.18" size="1.778" layer="95"/>
+</segment>
+<segment>
+<pinref part="U1" gate="G$2" pin="AGND"/>
+<wire x1="233.68" y1="83.82" x2="241.3" y2="83.82" width="0.1524" layer="91"/>
+<label x="241.3" y="83.82" size="1.778" layer="95"/>
+</segment>
+<segment>
+<pinref part="U1" gate="G$2" pin="CN10_GND"/>
+<wire x1="233.68" y1="81.28" x2="241.3" y2="81.28" width="0.1524" layer="91"/>
+<label x="241.3" y="81.28" size="1.778" layer="95"/>
+</segment>
+<segment>
+<pinref part="U1" gate="G$3" pin="CN6_GND"/>
+<wire x1="238.76" y1="48.26" x2="246.38" y2="48.26" width="0.1524" layer="91"/>
+<label x="246.38" y="48.26" size="1.778" layer="95"/>
+</segment>
+<segment>
+<pinref part="U1" gate="G$6" pin="CN5_GND"/>
+<wire x1="124.46" y1="17.78" x2="132.08" y2="17.78" width="0.1524" layer="91"/>
+<label x="132.08" y="17.78" size="1.778" layer="95"/>
+</segment>
+<segment>
+<pinref part="RESET" gate="-1" pin="S"/>
+<wire x1="81.28" y1="134.62" x2="83.82" y2="134.62" width="0.1524" layer="91"/>
+<label x="83.82" y="134.62" size="1.778" layer="95"/>
 </segment>
 </net>
@@
 </segment>
 </net>
+<net name="N$1" class="0">
+<segment>
+<pinref part="BATTERIE" gate="-2" pin="S"/>
+<pinref part="C1" gate="G$1" pin="1"/>
+<wire x1="22.86" y1="60.96" x2="27.94" y2="60.96" width="0.1524" layer="91"/>
+<pinref part="IC1" gate="A1" pin="VI"/>
+<wire x1="27.94" y1="60.96" x2="35.56" y2="60.96" width="0.1524" layer="91"/>
+<junction x="27.94" y="60.96"/>
+</segment>
+</net>
+<net name="N$4" class="0">
+<segment>
+<pinref part="RESET" gate="-2" pin="S"/>
+<pinref part="U1" gate="G$1" pin="CN7_RESET"/>
+<wire x1="106.68" y1="137.16" x2="81.28" y2="137.16" width="0.1524" layer="91"/>
+</segment>
+</net>

Commit message: gerber file for IA V2 + new libraries from mouser + Lidar / Ia / Asserv shield project creation
Parts:
- added R1, R2: (no value), rcl:R-EU_0204/7
Connections:
- net 5V: now also R1.2, R2.2
- net SCL: now also R2.1
- net SDA: now also R1.1
Changed lines of the file:
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@@
 <part name="C2" library="capacitor-wima" library_urn="urn:adsk.eagle:library:116" deviceset="C" device="5/2.5" value="0.1uF"/>
 <part name="RESET" library="con-molex" library_urn="urn:adsk.eagle:library:165" deviceset="22-23-2021" device=""/>
+<part name="R1" library="rcl" library_urn="urn:adsk.eagle:library:334" deviceset="R-EU_" device="0204/7" package3d_urn="urn:adsk.eagle:package:23498/1"/>
+<part name="R2" library="rcl" library_urn="urn:adsk.eagle:library:334" deviceset="R-EU_" device="0204/7" package3d_urn="urn:adsk.eagle:package:23498/1"/>
 </parts>
 <sheets>
@@
 <attribute name="NAME" x="76.2" y="137.922" size="1.524" layer="95" rot="R180"/>
 </instance>
+<instance part="R1" gate="G$1" x="99.06" y="114.3" smashed="yes" rot="R90">
+<attribute name="NAME" x="97.5614" y="110.49" size="1.778" layer="95" rot="R90"/>
+<attribute name="VALUE" x="102.362" y="110.49" size="1.778" layer="96" rot="R90"/>
+</instance>
+<instance part="R2" gate="G$1" x="190.5" y="111.76" smashed="yes" rot="R90">
+<attribute name="NAME" x="189.0014" y="107.95" size="1.778" layer="95" rot="R90"/>
+<attribute name="VALUE" x="193.802" y="107.95" size="1.778" layer="96" rot="R90"/>
+</instance>
 </instances>
 <busses>
@@
 <segment>
 <pinref part="U1" gate="G$1" pin="PB7"/>
-<wire x1="106.68" y1="109.22" x2="93.98" y2="109.22" width="0.1524" layer="91"/>
+<wire x1="106.68" y1="109.22" x2="99.06" y2="109.22" width="0.1524" layer="91"/>
 <label x="93.98" y="109.22" size="1.778" layer="95"/>
+<pinref part="R1" gate="G$1" pin="1"/>
+<wire x1="99.06" y1="109.22" x2="93.98" y2="109.22" width="0.1524" layer="91"/>
+<junction x="99.06" y="109.22"/>
 </segment>
 </net>
@@
 <segment>
 <pinref part="U1" gate="G$2" pin="PB6"/>
-<wire x1="198.12" y1="106.68" x2="185.42" y2="106.68" width="0.1524" layer="91"/>
+<wire x1="198.12" y1="106.68" x2="190.5" y2="106.68" width="0.1524" layer="91"/>
 <label x="185.42" y="106.68" size="1.778" layer="95"/>
+<pinref part="R2" gate="G$1" pin="1"/>
+<wire x1="190.5" y1="106.68" x2="185.42" y2="106.68" width="0.1524" layer="91"/>
+<junction x="190.5" y="106.68"/>
 </segment>
 <segment>
@@
 <junction x="63.5" y="60.96"/>
 <label x="73.66" y="60.96" size="1.778" layer="95"/>
+</segment>
+<segment>
+<pinref part="R1" gate="G$1" pin="2"/>
+<wire x1="99.06" y1="119.38" x2="99.06" y2="121.92" width="0.1524" layer="91"/>
+<label x="99.06" y="121.92" size="1.778" layer="95"/>
+</segment>
+<segment>
+<pinref part="R2" gate="G$1" pin="2"/>
+<wire x1="190.5" y1="116.84" x2="190.5" y2="119.38" width="0.1524" layer="91"/>
+<label x="190.5" y="119.38" size="1.778" layer="95"/>
 </segment>
 </net>
@@
 packages will not be understood (or retained) with this version.
 </note>
+<note version="8.4" severity="warning">
+Since Version 8.4, EAGLE supports properties for SPICE simulation.
+Probes in schematics and SPICE mapping objects found in parts and library devices
+will not be understood with this version. Update EAGLE to the latest version
+for full support of SPICE simulation.
+</note>
 </compatibility>
