File: AsservPami/asserv-pami.brd (EAGLE design)
At the start: 69.5 x 81.3 mm, 33 parts, among them IC1 NUCLEO-G431KB, IC2 7805TV

Commit message: fix name
Parts:
- renumbered ESP32-S3-ZERO-1 to ESP32-C3-ZERO-1, ESP32-S3-ZERO-2 to ESP32-C3-ZERO-2
Changed lines of the file:
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@@
 <attribute name="VALUE" x="49.53" y="37.338" size="0.6096" layer="27" font="vector" ratio="20"/>
 </element>
-<element name="ESP32-S3-ZERO-2" library="SparkFun-Connectors" library_urn="urn:adsk.eagle:library:513" package="1X09_LONGPADS" package3d_urn="urn:adsk.eagle:package:38155/2" value="" x="20.32" y="57.15" smashed="yes" rot="R90">
+<element name="ESP32-C3-ZERO-2" library="SparkFun-Connectors" library_urn="urn:adsk.eagle:library:513" package="1X09_LONGPADS" package3d_urn="urn:adsk.eagle:package:38155/2" value="" x="20.32" y="57.15" smashed="yes" rot="R90">
 <attribute name="NAME" x="18.161" y="56.134" size="0.6096" layer="25" font="vector" ratio="20" rot="R90"/>
 <attribute name="VALUE" x="23.114" y="56.134" size="0.6096" layer="27" font="vector" ratio="20" rot="R90"/>
 </element>
-<element name="ESP32-S3-ZERO-1" library="SparkFun-Connectors" library_urn="urn:adsk.eagle:library:513" package="1X09_LONGPADS" package3d_urn="urn:adsk.eagle:package:38155/2" value="" x="5.08" y="77.47" smashed="yes" rot="R270">
+<element name="ESP32-C3-ZERO-1" library="SparkFun-Connectors" library_urn="urn:adsk.eagle:library:513" package="1X09_LONGPADS" package3d_urn="urn:adsk.eagle:package:38155/2" value="" x="5.08" y="77.47" smashed="yes" rot="R270">
 <attribute name="NAME" x="7.239" y="78.486" size="0.6096" layer="25" font="vector" ratio="20" rot="R270"/>
 <attribute name="VALUE" x="2.286" y="78.486" size="0.6096" layer="27" font="vector" ratio="20" rot="R270"/>
@@
 <contactref element="POLOLU-U3V40F12" pad="2"/>
 <contactref element="POLOLU-U3V40F12" pad="3"/>
-<contactref element="ESP32-S3-ZERO-1" pad="2"/>
+<contactref element="ESP32-C3-ZERO-1" pad="2"/>
 <contactref element="I2C" pad="4"/>
 <contactref element="TIRETTE" pad="2"/>
@@
 <signal name="IA-TX">
 <contactref element="IC1" pad="1"/>
-<contactref element="ESP32-S3-ZERO-2" pad="8"/>
+<contactref element="ESP32-C3-ZERO-2" pad="8"/>
 <wire x1="20.32" y1="74.93" x2="24.13" y2="74.93" width="1.016" layer="1"/>
 <wire x1="24.13" y1="74.93" x2="25.4" y2="73.66" width="1.016" layer="1"/>
@@
 <signal name="IA-RX">
 <contactref element="IC1" pad="2"/>
-<contactref element="ESP32-S3-ZERO-2" pad="9"/>
+<contactref element="ESP32-C3-ZERO-2" pad="9"/>
 <wire x1="20.32" y1="77.47" x2="26.78894375" y2="77.47" width="1.016" layer="1"/>
 <wire x1="29.4629" y1="74.79604375" x2="29.4629" y2="72.52395625" width="1.016" layer="1"/>
@@
 <contactref element="IC2" pad="3"/>
 <contactref element="C2" pad="1"/>
-<contactref element="ESP32-S3-ZERO-1" pad="1"/>
+<contactref element="ESP32-C3-ZERO-1" pad="1"/>
 <contactref element="I2C" pad="3"/>
 <contactref element="R-5K1" pad="2"/>
@@
 <wire x1="24.2316" y1="52.55396875" x2="25.4" y2="53.72236875" width="1.016" layer="1"/>
 <wire x1="25.4" y1="60.96" x2="24.13" y2="62.23" width="1.016" layer="1"/>
-<contactref element="ESP32-S3-ZERO-2" pad="3"/>
+<contactref element="ESP32-C3-ZERO-2" pad="3"/>
 <wire x1="24.13" y1="62.23" x2="20.32" y2="62.23" width="1.016" layer="1"/>
 </signal>
@@
 <wire x1="23.0632" y1="53.0379375" x2="24.13" y2="54.1047375" width="1.016" layer="1"/>
 <wire x1="24.13" y1="58.42" x2="22.86" y2="59.69" width="1.016" layer="1"/>
-<contactref element="ESP32-S3-ZERO-2" pad="2"/>
+<contactref element="ESP32-C3-ZERO-2" pad="2"/>
 <wire x1="22.86" y1="59.69" x2="20.32" y2="59.69" width="1.016" layer="1"/>
 </signal>
@@
 <wire x1="6.35" y1="49.53" x2="10.16" y2="53.34" width="1.016" layer="16"/>
 <wire x1="10.16" y1="53.34" x2="10.16" y2="68.58" width="1.016" layer="16"/>
-<contactref element="ESP32-S3-ZERO-1" pad="4"/>
+<contactref element="ESP32-C3-ZERO-1" pad="4"/>
 <wire x1="10.16" y1="68.58" x2="8.89" y2="69.85" width="1.016" layer="16"/>
 <wire x1="8.89" y1="69.85" x2="5.08" y2="69.85" width="1.016" layer="16"/>
@@
 <wire x1="5.08" y1="51.18236875" x2="8.89" y2="54.99236875" width="1.016" layer="16"/>
 <wire x1="8.89" y1="54.99236875" x2="8.89" y2="66.04" width="1.016" layer="16"/>
-<contactref element="ESP32-S3-ZERO-1" pad="5"/>
+<contactref element="ESP32-C3-ZERO-1" pad="5"/>
 <wire x1="8.89" y1="66.04" x2="7.62" y2="67.31" width="1.016" layer="16"/>
 <wire x1="7.62" y1="67.31" x2="5.08" y2="67.31" width="1.016" layer="16"/>
@@
 <wire x1="3.81" y1="52.07" x2="7.62" y2="55.88" width="1.016" layer="16"/>
 <wire x1="7.62" y1="55.88" x2="7.62" y2="63.5" width="1.016" layer="16"/>
-<contactref element="ESP32-S3-ZERO-1" pad="6"/>
+<contactref element="ESP32-C3-ZERO-1" pad="6"/>
 <wire x1="7.62" y1="63.5" x2="6.35" y2="64.77" width="1.016" layer="16"/>
 <wire x1="6.35" y1="64.77" x2="5.08" y2="64.77" width="1.016" layer="16"/>
@@
 <wire x1="2.54" y1="8.89" x2="2.54" y2="60.96" width="1.016" layer="1"/>
 <wire x1="7.62" y1="3.81" x2="2.54" y2="8.89" width="1.016" layer="1"/>
-<contactref element="ESP32-S3-ZERO-1" pad="7"/>
+<contactref element="ESP32-C3-ZERO-1" pad="7"/>
 <wire x1="2.54" y1="60.96" x2="3.81" y2="62.23" width="1.016" layer="1"/>
 <wire x1="3.81" y1="62.23" x2="5.08" y2="62.23" width="1.016" layer="1"/>
@@
 <wire x1="20.32" y1="41.91" x2="15.24" y2="41.91" width="1.016" layer="1"/>
 <wire x1="15.24" y1="41.91" x2="15.24" y2="58.42" width="1.016" layer="1"/>
-<contactref element="ESP32-S3-ZERO-1" pad="8"/>
+<contactref element="ESP32-C3-ZERO-1" pad="8"/>
 <wire x1="15.24" y1="58.42" x2="13.97" y2="59.69" width="1.016" layer="1"/>
 <wire x1="13.97" y1="59.69" x2="5.08" y2="59.69" width="1.016" layer="1"/>
@@
 <wire x1="13.97" y1="35.56" x2="12.7" y2="36.83" width="1.016" layer="1"/>
 <wire x1="12.7" y1="36.83" x2="12.7" y2="55.88" width="1.016" layer="1"/>
-<contactref element="ESP32-S3-ZERO-1" pad="9"/>
+<contactref element="ESP32-C3-ZERO-1" pad="9"/>
 <wire x1="12.7" y1="55.88" x2="11.43" y2="57.15" width="1.016" layer="1"/>
 <wire x1="11.43" y1="57.15" x2="5.08" y2="57.15" width="1.016" layer="1"/>
@@
 <signal name="N$5">
 <contactref element="UART" pad="1"/>
-<contactref element="ESP32-S3-ZERO-2" pad="4"/>
+<contactref element="ESP32-C3-ZERO-2" pad="4"/>
 <wire x1="8.89" y1="39.37" x2="13.97" y2="39.37" width="1.016" layer="16"/>
 <wire x1="13.97" y1="39.37" x2="13.97" y2="64.77" width="1.016" layer="16"/>
@@
 <signal name="N$6">
 <contactref element="UART" pad="2"/>
-<contactref element="ESP32-S3-ZERO-2" pad="5"/>
+<contactref element="ESP32-C3-ZERO-2" pad="5"/>
 <wire x1="20.32" y1="67.31" x2="11.43" y2="67.31" width="1.016" layer="16"/>
 <wire x1="11.43" y1="67.31" x2="11.3284" y2="67.2084" width="1.016" layer="16"/>

Commit message: fix pami woard
Parts:
- added R-5K5, R-5K6: (no value), rcl:0204/7
- C1: value 0.33uF -> 0.1uF
- C2: value 0.1uF -> 22uF
- C3: value 0.33uF -> 33uF
- IC2: value 7805TV -> L4941BV
- moved CODEUR1 14.0 mm to (63.5, 33.0)
- moved CODEUR2 14.0 mm to (54.6, 33.0)
- moved C3 12.7 mm to (55.9, 54.6)
- moved POLOLU-U3V40F12 12.7 mm to (50.8, 52.1)
Connections:
- net 5V: now also R-5K5.2, R-5K6.2; no longer IC1.27
- net SCL: now also R-5K6.1
- net SDA: now also R-5K5.1
- net VIN: now also IC1.30
Routing:
- net 5V: track 177.3 -> 216.6 mm, vias 2 -> 1
- net ENC1-B: track 26.0 -> 41.3 mm
- net ENC2-A: track 13.5 -> 27.3 mm
- net 12V: track 61.1 -> 73.8 mm, vias 0 -> 1
- net ENC1-A: track 54.0 -> 65.8 mm, vias 0 -> 2
- net ENC2-B: track 10.7 -> 22.2 mm
- net SCL: track 20.1 -> 28.2 mm
- net VIN: track 64.3 -> 68.7 mm, vias 0 -> 1
- net SDA: track 27.0 -> 30.8 mm
- net N$5: track 36.8 -> 39.7 mm
- net PWM-1-2: track 56.0 -> 53.7 mm
- net IA-RX: track 14.6 -> 12.5 mm
- net SENSE-2: track 43.5 -> 44.5 mm
- net PWM-1-1: track 49.8 -> 49.1 mm
- net SERVO1: track 36.6 -> 37.4 mm
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