File: KiCad/pami-board/pami-board.kicad_pcb (KiCad board)
At the start: 4 copper layers, 73.4 x 80 mm, 38 parts, among them J1 Nucleo-G431KB, J10 Codeur1, J11 Codeur2, J12 SRF04, J13 Servo, J14 Connector, USB-TYPE-C-16P, J15 Motor-MP6550-1, J16 Motor-MP6550-1, J17 Motor-MP6550-2, J18 Motor-MP6550-2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

Commit message: fix alimentation 12V et USB
Connections:
- C1 pad 1: Net-(J8-Pin_1) -> +12V
- C3 pad 1: Net-(J8-Pin_1) -> +12V
- F1 pad 1: +12V -> Net-(J7-Pin_1)
- J14 pad B6: unconnected-(J14-D+-PadB6) -> USB-D+
- J14 pad B7: unconnected-(J14-D--PadB7) -> USB-D-
- J7 pad 1: +12V -> Net-(J7-Pin_1)
- J8 pad 1: Net-(J8-Pin_1) -> +12V
- J9 pad 1: Net-(J8-Pin_1) -> +12V
- R1 pad 1: Net-(J8-Pin_1) -> +12V
- U1 pad 2: Net-(J8-Pin_1) -> +12V
Routing:
- net Net-(J8-Pin_1): track 38.5 -> 0.00 mm, vias 1 -> 0
- net +12V: track 133.9 -> 160.8 mm, vias 0 -> 1
- net Net-(J7-Pin_1): track 0.00 -> 18.6 mm
- net USB-D+: track 13.2 -> 22.1 mm
- net USB-D-: track 36.2 -> 40.3 mm, vias 0 -> 2
