File: KiCad/pami-board/pami-board.kicad_sch (KiCad schematic)
At the start: 38 parts, among them J1 Nucleo-G431KB, J10 Codeur1, J11 Codeur2, J12 SRF04, J13 Servo, J14 Connector, USB-TYPE-C-16P, J15 Motor-MP6550-1, J16 Motor-MP6550-1, J17 Motor-MP6550-2, J18 Motor-MP6550-2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

Commit message: fix alimentation 12V et USB
Connections:
- net +12V: now also C1.1, C3.1, J8.1 (Pin_1), J9.1 (Pin_1), R1.1, U1.2 (VIN); no longer F1.1, J7.1 (Pin_1)
- net USB-D+: now also J14.B6 (D+)
- net USB-D-: now also J14.B7 (D-)
- new net: F1.1, J7.1 (Pin_1)
Changed lines of the file:
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@@
 	)
 	(junction
-		(at 21.59 171.45)
-		(diameter 0)
-		(color 0 0 0 0)
-	)
-	(junction
 		(at 135.89 161.29)
 		(diameter 0)
@@
 	(wire
 		(pts
+			(xy 224.79 41.91) (xy 224.79 44.45)
+		)
+		(stroke
+			(width 0)
+			(type default)
+		)
+	)
+	(wire
+		(pts
 			(xy 81.28 110.49) (xy 83.82 110.49)
 		)
@@
 	(wire
 		(pts
+			(xy 39.37 171.45) (xy 39.37 175.26)
+		)
+		(stroke
+			(width 0)
+			(type default)
+		)
+	)
+	(wire
+		(pts
 			(xy 210.82 95.25) (xy 229.87 95.25)
 		)
@@
 	(wire
 		(pts
-			(xy 227.33 74.93) (xy 229.87 74.93)
+			(xy 219.71 41.91) (xy 219.71 44.45)
 		)
 		(stroke
@@
 	(wire
 		(pts
-			(xy 260.35 80.01) (xy 264.16 80.01)
+			(xy 227.33 74.93) (xy 229.87 74.93)
 		)
 		(stroke
@@
 	(wire
 		(pts
-			(xy 147.32 161.29) (xy 154.94 161.29)
+			(xy 260.35 80.01) (xy 264.16 80.01)
 		)
 		(stroke
@@
 	(wire
 		(pts
-			(xy 224.79 140.97) (xy 227.33 140.97)
+			(xy 147.32 161.29) (xy 154.94 161.29)
 		)
 		(stroke
@@
 	(wire
 		(pts
-			(xy 224.79 124.46) (xy 227.33 124.46)
+			(xy 224.79 140.97) (xy 227.33 140.97)
 		)
 		(stroke
@@
 	(wire
 		(pts
-			(xy 224.79 119.38) (xy 227.33 119.38)
+			(xy 224.79 124.46) (xy 227.33 124.46)
 		)
 		(stroke
@@
 	(wire
 		(pts
-			(xy 87.63 60.96) (xy 90.17 60.96)
+			(xy 224.79 119.38) (xy 227.33 119.38)
 		)
 		(stroke
@@
 	(wire
 		(pts
-			(xy 81.28 128.27) (xy 83.82 128.27)
+			(xy 87.63 60.96) (xy 90.17 60.96)
 		)
 		(stroke
@@
 	(wire
 		(pts
-			(xy 21.59 171.45) (xy 21.59 176.53)
+			(xy 81.28 128.27) (xy 83.82 128.27)
 		)
 		(stroke
@@
 		)
 	)
+	(global_label "USB-D+"
+		(shape input)
+		(at 219.71 44.45 270)
+		(fields_autoplaced yes)
+		(effects
+			(font
+				(size 1.27 1.27)
+			)
+			(justify right)
+		)
+		(property "Intersheetrefs" "${INTERSHEET_REFS}"
+			(at 219.71 55.66 90)
+			(effects
+				(font
+					(size 1.27 1.27)
+				)
+				(justify right)
+				(hide yes)
+			)
+		)
+	)
 	(global_label "ENC2-A"
 		(shape input)
@@
 		)
 	)
+	(global_label "USB-D-"
+		(shape input)
+		(at 224.79 44.45 270)
+		(fields_autoplaced yes)
+		(effects
+			(font
+				(size 1.27 1.27)
+			)
+			(justify right)
+		)
+		(property "Intersheetrefs" "${INTERSHEET_REFS}"
+			(at 224.79 55.66 90)
+			(effects
+				(font
+					(size 1.27 1.27)
+				)
+				(justify right)
+				(hide yes)
+			)
+		)
+	)
 	(global_label "BST"
 		(shape input)
@@
 	(symbol
 		(lib_id "power:+12V")
-		(at 21.59 176.53 180)
+		(at 39.37 175.26 180)
 		(unit 1)
 		(exclude_from_sim no)
@@
 		(fields_autoplaced yes)
 		(property "Reference" "#PWR012"
-			(at 21.59 172.72 0)
+			(at 39.37 171.45 0)
 			(effects
 				(font
@@
 		)
 		(property "Value" "+12V"
-			(at 21.59 181.61 0)
+			(at 39.37 180.34 0)
 			(effects
 				(font
@@
 		)
 		(property "Footprint" ""
-			(at 21.59 176.53 0)
+			(at 39.37 175.26 0)
 			(effects
 				(font
@@
 		)
 		(property "Datasheet" ""
-			(at 21.59 176.53 0)
+			(at 39.37 175.26 0)
 			(effects
 				(font
@@
 		)
 		(property "Description" "Power symbol creates a global label with name \"+12V\""
-			(at 21.59 176.53 0)
+			(at 39.37 175.26 0)
 			(effects
 				(font
