File: KiCad/balise-tofs/balise-tofs.kicad_sch (KiCad schematic)
At the start: 97 parts, among them J1 Vin, J10 Conn_02x05_Odd_Even, J11 Conn_02x05_Odd_Even, J12 Conn_02x05_Odd_Even, J13 Conn_02x05_Odd_Even, J14 Conn_02x05_Odd_Even, J15 Conn_02x05_Odd_Even, J16 Conn_02x05_Odd_Even, J17 Conn_02x05_Odd_Even, J18 Conn_02x05_Odd_Even, J19 Conn_02x05_Odd_Even, J2 Conn_01x03, J20 Conn_02x05_Odd_Even, J21 Conn_02x05_Odd_Even, Q1 Q_PMOS_GDS, U1 AP63203WU-7, U2 NUCLEO-G431KB, U3 PCA9535CPW, U4 AP63205WU-7, U5 74AHCT1G125

Commit message: finalisation du routage
Parts:
- added R20, R21, R22, R23: 2.2k, Resistor_SMD:R_0603_1608Metric, symbol Device:R
- C1: LCSC (none) -> C165580
- C11, C12, C36, C37: LCSC (none) -> C52306
- C2, C3, C35, C5: LCSC (none) -> C138687
- C20, C21, C22, C23, C24, C25, C26, C27, C28, C29, C30, C31: LCSC (none) -> C15850
- C33, C34, C39, C4, C40, C41, C42, C43, C44, C45, C46, C47, C48, C49, C50, C51, C6, C7: LCSC (none) -> C14663
- C38: LCSC (none) -> C165531
- D1: LCSC (none) -> C173427
- D2: LCSC C19077578 -> C151920
- D3: LCSC (none) -> C2986059
- D4: LCSC (none) -> C2286
- J1: LCSC (none) -> C158012
- J2: LCSC (none) -> C144394
- L1: LCSC (none) -> C15269
- L2: LCSC (none) -> C57269
- Q1: value Q_PMOS_GDS -> SI2307A; LCSC (none) -> C347490
- R1, R32: LCSC (none) -> C25803
- R2, R3: LCSC (none) -> C21190
- R33: value 16k -> 15k; LCSC (none) -> C22809
- R34: LCSC (none) -> C25804
- R40, R41, R42, R43, R44, R45, R46, R47, R48, R49, R50, R51, R60, R61, R62, R63, R64, R65, R66, R67, R68, R69, R70, R71: LCSC (none) -> C22775
- R80: LCSC (none) -> C23138
- U1: LCSC (none) -> C780769
- U3: LCSC (none) -> C2652292
- U4: LCSC (none) -> C2071056
- U5: LCSC (none) -> C7484
Connections:
- net 3V3_SENS: now also R20.2, R21.2, R22.2, R23.2
- net SCL_A: now also R21.1
- net SCL_B: now also R23.1
- net SDA_A: now also R20.1
- net SDA_B: now also R22.1

Commit message: Mise dans le bon sens du TVS D2 SMBJ22A sur le rail d'alimentation monté à l'envers Réglage de l'inductance à 3.9µH (au lieu de 3.3) du rail d'alimentation 3.3v comme indiqué dans la fiche technique https://www.diodes.com/assets/Datasheets/AP63200-AP63201-AP63203-AP63205.pdf Alimentation de la nucleo en 5v via son rail 5V CN3_4 à partir du rail 5v Remplissage du cartouche du schéma
Parts:
- L1: value 3.3uH -> 3.9uH
Connections:
- net 5V: now also U2.CN3_4 (5V)
- net GND: now also D2.2; no longer D2.1
- net VBAT: now also D2.1; no longer D2.2
Other:
- company: (none) -> ESIALROBOTIK
- title: (none) -> Balise de détection ToF
- moved on the sheet: D2
Changed lines of the file:
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@@
 	(generator_version "10.0")
 	(paper "A3")
+	(title_block
+		(title "Balise de détection ToF")
+		(date "2026-10-16")
+		(rev "0.2")
+		(company "ESIALROBOTIK")
+	)
 	(junction
 		(at 269.24 40.64)
@@
 	(wire
 		(pts
+			(xy 93.98 118.11) (xy 90.17 118.11)
+		)
+		(stroke
+			(width 0)
+			(type default)
+		)
+	)
+	(wire
+		(pts
 			(xy 375.92 146.05) (xy 375.92 153.67)
 		)
@@
 		)
 	)
+	(global_label "5V"
+		(shape input)
+		(at 93.98 118.11 0)
+		(fields_autoplaced yes)
+		(effects
+			(font
+				(size 1.27 1.27)
+			)
+			(justify left)
+		)
+		(property "Intersheetrefs" "${INTERSHEET_REFS}"
+			(at 99.2633 118.11 0)
+			(hide yes)
+			(show_name no)
+			(do_not_autoplace no)
+			(effects
+				(font
+					(size 1.27 1.27)
+				)
+				(justify left)
+			)
+		)
+	)
 	(global_label "3V3_SENS"
 		(shape input)
@@
 			)
 		)
-		(property "Value" "3.3uH"
+		(property "Value" "3.9uH"
 			(at 265.43 38.1 90)
 			(show_name no)
@@
 	(symbol
 		(lib_id "PCM_JLCPCB-Diodes:TVS-Uni,SMBJ24A")
-		(at 74.93 45.72 0)
+		(at 74.93 45.72 180)
 		(unit 1)
 		(body_style 1)
@@
 		(fields_autoplaced yes)
 		(property "Reference" "D2"
-			(at 78.74 44.7674 0)
+			(at 78.74 44.1324 0)
 			(show_name no)
 			(do_not_autoplace no)
@@
 					(size 1.27 1.27)
 				)
-				(justify left)
+				(justify right)
 			)
 		)
 		(property "Value" "SMBJ22A"
-			(at 78.74 47.3075 0)
+			(at 78.74 46.6725 0)
 			(show_name no)
 			(do_not_autoplace no)
@@
 					(size 0.8 0.8)
 				)
-				(justify left)
+				(justify right)
 			)
 		)
 		(property "Footprint" "PCM_JLCPCB:D_SMB"
-			(at 73.152 45.72 90)
+			(at 76.708 45.72 90)
 			(hide yes)
 			(show_name no)

Commit message: dernières mise à jour avant production
Parts:
- added D5: D_Schottky, Diode_SMD:D_SOD-123, symbol Device:D_Schottky
- added J22: Cavalier, Connector_JST:JST_XH_B2B-XH-A_1x02_P2.50mm_Vertical, symbol Connector_Generic:Conn_01x02
Connections:
- net 5V: now also D5.2 (A); no longer U2.CN3_4 (5V)
- new net: J22.2 (Pin_2), U2.CN3_4 (5V)
- new net: D5.1 (K), J22.1 (Pin_1)
- no-connect marks 74 -> 73
Other:
- moved on the sheet: D3, D4, R2, R3
